File: hardware/openpod-1/openpod-1.sch (KiCad schematic (older format))
At the start: 78 parts, among them J1 USB_B_Micro, J2 AudioJack2_Ground, J3 Micro_SD_Card, Q1 TRANSISTOR_NPNSOT23-3, SW1 SW_Push, U1 MCP73831-2-OT, U2 SPX3819M5-L-3-3, U3 click-wheel, U4 ATSAMD21G18A-AUT, U5 AT42QT2120_COMMS, U6 VS1053B, U7 VREG_SOT23-6_DUALAP7312, X2 JSTPH, Y1 ABM8G-12.288MHZ-18-D2Y-T, Y2 Crystal

Commit message: update click wheel, use connectors
Parts:
- removed LCD1: JD-T1800, little-helper:JD-T1800, symbol little-helper:JD-T1800
- removed Q1: TRANSISTOR_NPNSOT23-3, little-helper:SOT23-3, symbol little-helper:TRANSISTOR_NPNSOT23-3
- added Q1: 220mA/50V/3.5Ω, sparkfun:SOT23-3, symbol sparkfun:MOSFET-NCH-BSS138
- added R28: 1, Resistor_SMD:R_0805_2012Metric, symbol Device:R
- added R29, R30, R31: 1k, Resistor_SMD:R_0402_1005Metric, symbol Device:R
- added R9: 10k, Resistor_SMD:R_0805_2012Metric, symbol Device:R
- added U8: KWH018ST14-F01_4WSPI-TOP, sparkfun:FPC05040-17204, symbol sparkfun:KWH018ST14-F01_4WSPI-TOP
- D1: MFR (none) -> MBR120VLSFT3G; Mouser (none) -> 863-MBR120VLSFT3G
- FB1, FB2: Mouser (none) -> BLM21SP181SH1D
- J1: MFR (none) -> 47346-0001; Mouser (none) -> 538-47346-0001
- J2: footprint custom:Jack_3.5mm_CUI_SJ-3523-SMT_Horizontal-G -> Connector_Audio:Jack_3.5mm_CUI_SJ-3524-SMT_Horizontal; MFR (none) -> SJ-3523-SMT-TR; Mouser (none) -> 490-SJ-3523-SMT-TR
- J3: MFR (none) -> DM3D-SF; Mouser (none) -> 798-DM3D-SF
- R14: value 22 -> 10k
- R15: value 1k -> 1
- S1: Field4 Wurth Electronics -> (none); Field5 Unavailable -> (none); Field6 None -> (none); Field7 450302014072 -> (none); Field8 SWITCH, SLIDE, MINI, ON-ON, RIGHT ANGLE; Contact Configurat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 -> (none); MFR (none) -> 450302014072; Mouser (none) -> 710-450302014072
- U1: MFR (none) -> MCP73831T-2ACI/OT; Mouser (none) -> 579-MCP73831T-2ACIOT
- U2: MFR (none) -> SPX3819M5-L-5-0/TR; Mouser (none) -> 701-SPX3819M5-L-50TR
- U4: mouser (none) -> 556-ATSAMD21G18A-AUT
- U5: MFR (none) -> AT42QT2120-SUR; Mouser (none) -> 556-AT42QT2120-SUR
- U6: Field4 VS1053B -> (none); Field5 None -> (none); Field6 Adafruit Industries -> (none); Field7 None -> (none); Field8 SMD IC Codecoder; -> (none); Mouser (none) -> 485-1681
- U7: value VREG_SOT23-6_DUALAP7312 -> TLV733P-Q1; MFR (none) -> TLV73318PQDBVRQ1; Mouser (none) -> 595-TLV73318PQDBVRQ1
- X2: MFR (none) -> S2B-PH-SM4-TB(LF)(SN)
- Y1: Field4 ABM8G-12.288MHZ-18-D2Y-T -> (none); Field5 SMD-4 Abracon -> (none); Field6 Abracon -> (none); Field7 None -> (none); Field8 Crystal 12.288MHz ±20ppm _Tol_ ±30ppm _Stability_ 18pF FUND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 -> (none); MFR (none) -> ABM8G-12.288MHZ-18-D2Y-T; Mouser (none) -> 815-ABM8G-12.2-18D2Y
Connections:
- net +3V3: now also R14.1, R9.1, U8.P$10 (P68), U8.P$15 (RD/E), U8.P$35 (IOVCC), U8.P$36 (VCC), U8.P$37 (~RST), U8.P$40 (LEDA)
- net D11: now also R9.2, U8.P$12 (~CS)
- net D12: now also U8.P$14 (WR/RW)
- net D13: now also R28.1; no longer R15.1
- net Earth: now also Q1.2 (S), U8.P$1 (GND), U8.P$11 (SPI4W), U8.P$17 (GND), U8.P$18 (GND), U8.P$19 (GND), U8.P$20 (GND), U8.P$21 (GND), U8.P$22 (GND), U8.P$23 (GND), U8.P$24 (GND), U8.P$25 (GND), U8.P$26 (GND), U8.P$27 (GND), U8.P$28 (GND), U8.P$29 (GND), U8.P$30 (GND), U8.P$31 (GND), U8.P$32 (GND), U8.P$33 (GND), U8.P$38 (GND), U8.P$6 (GND), U8.P$7 (IM0), U8.P$8 (IM1), U8.P$9 (IM2)
- net MOSI: now also U8.P$16 (DB0/SDI)
- net SCK: now also U8.P$13 (DC/SCL)
- net LEDK: now reaches R14.2
- net LEDK: now also Q1.1 (G), U8.P$39 (LEDK)
- net at R15.2: now also Q1.3 (D)
- net at R27.2: now also U3.7; no longer U3.4
- net at R26.2: now also U3.6; no longer U3.3
- net at R25.2: now also U3.5; no longer U3.2
- net at R24.2: now also U3.4; no longer U3.1
- net at R23.2: now also U3.12; no longer U3.9
- net at R22.2: now also U3.11; no longer U3.8
- net at R21.2: now also U3.10; no longer U3.7
- net at U5.18 (KEY11/GPO9): now also R29.1
- net at U5.19 (KEY10/GPO8): now also R30.1
- net at U5.20 (KEY9/GPO7): now also R31.1
- net at R20.2: now also U3.9; no longer U3.6
- net at R19.2: now also U3.8; no longer U3.5
- new net: R31.2, U3.3
- new net: R30.2, U3.2
- new net: R29.2, U3.1
- new net: R15.1, R28.2
- no-connect marks 18 -> 17
Other:
- note added: "BACKLIGHT\n"
- note added: "SCREEN\n"
- note removed: "Screen"
- moved on the sheet: JP3, JP4, U3

Commit message: revision 1
Parts:
- removed J2: AudioJack2_Ground, Connector_Audio:Jack_3.5mm_CUI_SJ-3524-SMT_Horizontal, symbol Connector:AudioJack2_Ground
- added H1, H2, H3: MountingHole, MountingHole:MountingHole_2.2mm_M2_DIN965_Pad, symbol Mechanical:MountingHole
- added HS1, HS2: Heatsink_Pad, custom:medium-thermal, symbol Mechanical:Heatsink_Pad
- added HS3: Heatsink_Pad, custom:thermal, symbol Mechanical:Heatsink_Pad
- added HS4: Heatsink_Pad, custom:small-thermal, symbol Mechanical:Heatsink_Pad
- added J2: SJ-3524-SMT-jack, Connector_Audio:Jack_3.5mm_CUI_SJ-3524-SMT_Horizontal, symbol jack:SJ-3524-SMT
- C19, C20: footprint Capacitor_THT:CP_Radial_D5.0mm_P2.00mm -> Capacitor_SMD:CP_Elec_6.3x5.4; Mouser Number (none) -> 667-EEE-0JA221WP; Reference (none) -> EEE-0JA221WP
- D1: MFR MBR120VLSFT3G -> (none); Mouser 863-MBR120VLSFT3G -> (none); Mouser Number (none) -> 863-MBR120VLSFT3G; Reference (none) -> MBR120VLSFT3G
- FB1, FB2: Mouser BLM21SP181SH1D -> (none); Mouser Number (none) -> BLM21SP181SH1D
- J1: MFR 47346-0001 -> (none); Mouser 538-47346-0001 -> (none); Mouser Number (none) -> 538-47346-0001; Reference (none) -> 47346-0001
- J3: MFR DM3D-SF -> (none); Mouser 798-DM3D-SF -> (none); Mouser Number (none) -> 798-DM3D-SF; Reference (none) -> DM3D-SF
- Q1: MFR BSS138 -> (none); Mouser 512-BSS138 -> (none); Mouser Number (none) -> 512-BSS138; Reference (none) -> BSS138
- S1: MFR 450302014072 -> (none); Mouser 710-450302014072 -> (none); Mouser Number (none) -> 710-450302014072; Reference (none) -> 450302014072
- SW1: footprint Button_Switch_SMD:SW_Push_SPST_NO_Alps_SKRK -> reset-button:PTS647; Mouser Number (none) -> 611-PTS647SM38SMTR2L; Reference (none) -> PTS647SM38SMTR2LFS
- U1: MFR MCP73831T-2ACI/OT -> (none); Mouser 579-MCP73831T-2ACIOT -> (none); Mouser Number (none) -> 579-MCP73831T-2ACIOT; Reference (none) -> MCP73831T-2ACI/OT
- U2: MFR SPX3819M5-L-5-0/TR -> (none); Mouser 701-SPX3819M5-L-50TR -> (none); Mouser Number (none) -> 701-SPX3819M5-L-50TR; Reference (none) -> SPX3819M5-L-5-0/TR
- U4: Mouser Number (none) -> 556-ATSAMD21G18A-AUT; mouser 556-ATSAMD21G18A-AUT -> (none)
- U5: MFR AT42QT2120-SUR -> (none); Mouser 556-AT42QT2120-SUR -> (none); Mouser Number (none) -> 556-AT42QT2120-SUR; Reference (none) -> AT42QT2120-SUR
- U6: Mouser 485-1681 -> (none); Mouser Number (none) -> 485-1681
- U7: MFR TLV73318PQDBVRQ1 -> (none); Mouser 595-TLV73318PQDBVRQ1 -> (none); Mouser Number (none) -> 595-TLV73318PQDBVRQ1; Reference (none) -> TLV73318PQDBVRQ1
- U8: MFR XF3M-4015-1B -> (none); Mouser 653-XF3M-4015-1B -> (none); Mouser Number (none) -> 653-XF3M-4015-1B; Reference (none) -> XF3M-4015-1B
- X2: footprint Connector_JST:JST_PH_S2B-PH-K_1x02_P2.00mm_Horizontal -> little-helper:JST-2-SMD; MFR S2B-PH-SM4-TB(LF)(SN) -> (none); Reference (none) -> S2B-PH-SM4-TB(LF)(SN)
- Y1: MFR ABM8G-12.288MHZ-18-D2Y-T -> (none); Mouser 815-ABM8G-12.2-18D2Y -> (none); Mouser Number (none) -> 815-ABM8G-12.2-18D2Y; Reference (none) -> ABM8G-12.288MHZ-18-D2Y-T
Connections:
- net AGND: now also J2.S
- net D8: now also U6.8 (DREQ)
- net D9: no longer U6.8 (DREQ)
- net Earth: now also HS2.1, HS3.1, HS4.1
- net L_OUT: now also J2.T
- net R_OUT: now also J2.R
- net VBUS: now also HS1.1
- no-connect marks 17 -> 18
Other:
- note added: "Mounting Holes"
